File: pcb/esp-gateway/esp-gateway.kicad_pcb (KiCad board)
At the start: 2 copper layers, 101.9 x 57.4 mm, 33 parts, among them J1 ESP-01, J10 JMP, J2 RF-TR, J3 RF-RX, J4 USB, J5 Conn_01x02, J6 Conn_01x02, J7 UART0, J8 Conn_01x02, J9 Conn_02x04_Counter_Clockwise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

Commit message: done
Parts:
- added G***: LOGO, LOGO, B.Cu at (134.2, 75.4)
- added REF**: PinHeader_1x04_P2.54mm_Vertical, Connector_PinHeader_2.54mm:PinHeader_1x04_P2.54mm_Vertical, B.Cu at (126.9, 90.6)
- AE1, AE2, AE3, AE4: value Antenna -> Antenna_Shield; footprint Connector_Coaxial:U.FL_Hirose_U.FL-R-SMT-1_Vertical -> Connector_Coaxial:U.FL_Molex_MCRF_73412-0110_Vertical
- turned AE1 to 90 degrees
- turned AE2 to -90 degrees
- turned AE3 to -90 degrees
- turned AE4 to 90 degrees
Connections:
- AE1 pad 2: (no net) -> GND
- AE2 pad 2: (no net) -> GND
- AE3 pad 2: (no net) -> GND
- AE4 pad 2: (no net) -> GND
Routing:
- net /SDA: track 43.5 -> 122.0 mm, vias 1 -> 2
- net /SCL: track 43.8 -> 117.1 mm, vias 1 -> 2
- net +5V: track 125.3 -> 129.6 mm
- net /DIO0-3: track 73.8 -> 72.3 mm, vias 0 -> 2
- net GND: vias 38 -> 41
Other:
- board text added: "3V3 5V SDA SCL + -"
- board text added: "BOOT0"
- board text added: "Designed by:"
- board text added: "ESP-01"
- board text added: "ESP32-S2-WROOM"
- board text added: "NRF24L01"
- board text added: "OLED"
- board text added: "PWR"
- board text added: "RESET"
- board text added: "RF-RX"
- board text added: "RF-TX"
- board text added: "UART0"
- board text added: "USB"
- board text added: "Universal ESP Gateway v1.0"
