File: pcb/esp-gateway/esp-gateway.kicad_sch (KiCad schematic)
At the start: 33 parts, among them J1 ESP-01, J10 JMP, J2 RF-TR, J3 RF-RX, J4 USB, J5 Conn_01x02, J6 Conn_01x02, J7 UART0, J8 Conn_01x02, J9 Conn_02x04_Counter_Clockwise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

Commit message: done
Parts:
- removed AE1, AE2, AE3, AE4: Antenna, Connector_Coaxial:U.FL_Hirose_U.FL-R-SMT-1_Vertical, symbol Device:Antenna
- added AE1, AE2, AE3, AE4: Antenna_Shield, Connector_Coaxial:U.FL_Molex_MCRF_73412-0110_Vertical, symbol Device:Antenna_Shield
Connections:
- net GND: now also AE1.2 (Shield), AE2.2 (Shield), AE3.2 (Shield), AE4.2 (Shield)
- net at U3.9 (ANT): now also AE1.1 (A)
- net at U2.1 (ANT): now also AE2.1 (A)
- net at U4.1 (ANT): now also AE3.1 (A)
- net at U5.9 (ANT): now also AE4.1 (A)
Other:
- moved on the sheet: U2, U3, U4
